Commit message: add cameras to robot model

File: wr8_description/urdf/model.urdf.xacro (robot description, xacro)
@@ -29,4 +29,10 @@
   <xacro:property name="servo_no_load_speed" value="4.553"/> -->
   <xacro:property name="wheel_friction" value="1.75" />
+  <!-- camera properties -->
+  <xacro:property name="cam_height" value="0.05"/>
+  <xacro:property name="cam_radius" value="0.02"/>
+  <xacro:property name="cam_mass" value="0.05"/>
+  <xacro:property name="base_link_lcam_xyz" value="0.14 0.15 0.18"/>
+  <xacro:property name="base_link_rcam_xyz" value="0.14 -0.15 0.18"/>
   <xacro:arg name="pub_tf" default="true" />
   <xacro:arg name="robot_name" default="robot" />
@@ -259,3 +265,70 @@
     </sensor>
   </gazebo>
+  <!-- camera macro -->
+  <xacro:macro name="single_camera" params="name base_link">
+    <link name="${name}_frame">
+      <xacro:solid_cylinder_inertial
+          r="${cam_radius}" h="${cam_height}"
+          mass="${cam_mass}" >
+        <origin xyz="0 0 0" rpy="0 ${degrees_90} 0" />
+      </xacro:solid_cylinder_inertial>
+      <collision>
+        <origin xyz="0 0 0" rpy="0 ${degrees_90} 0" />
+        <geometry>
+          <cylinder length="${cam_height}" radius="${cam_radius}"/>
+        </geometry>
+      </collision>
+      <visual>
+        <origin xyz="0 0 0" rpy="0 ${degrees_90} 0" />
+        <geometry>
+          <cylinder length="${cam_height}" radius="${cam_radius}"/>
+        </geometry>
+      </visual>
+    </link>
+    <joint name="${name}_joint" type="fixed">
+      <child link="${name}_frame" />
+      <parent link="base_link" />
+      <origin xyz="${base_link}" />
+    </joint>
+    <gazebo reference="${name}_frame">
+      <material>Gazebo/Black</material>
+      <sensor type="camera" name="${name}">
+        <!-- required FPS -->
+        <update_rate>15.0</update_rate>
+        <camera name="${name}">
+          <horizontal_fov>1.3962634</horizontal_fov>
+          <image>
+            <width>800</width>
+            <height>800</height>
+            <format>R8G8B8</format>
+          </image>
+          <clip>
+            <near>0.02</near>
+            <far>300</far>
+          </clip>
+          <noise>
+            <type>gaussian</type>
+            <mean>0.0</mean>
+            <stddev>0.007</stddev>
+        </noise>
+        </camera>
+        <plugin name="${name}_controller" filename="libgazebo_ros_camera.so">
+          <alwaysOn>true</alwaysOn>
+          <updateRate>0.0</updateRate>
+          <cameraName>$(arg robot_name)/${name}</cameraName>
+          <imageTopicName>cam_image_raw</imageTopicName>
+          <cameraInfoTopicName>cam_info</cameraInfoTopicName>
+          <frameName>lcam_frame</frameName>
+          <hackBaseline>0.07</hackBaseline>
+          <distortionK1>0.0</distortionK1>
+          <distortionK2>0.0</distortionK2>
+          <distortionK3>0.0</distortionK3>
+          <distortionT1>0.0</distortionT1>
+          <distortionT2>0.0</distortionT2>
+        </plugin>
+      </sensor>
+    </gazebo>
+  </xacro:macro>
+  <xacro:single_camera name="lcam" base_link="${base_link_lcam_xyz}" />
+  <xacro:single_camera name="rcam" base_link="${base_link_rcam_xyz}" />
 </robot>
